Commit message: update xacro

File: src/quaro_description/urdf/leg/leg.0.0.xacro (robot description, xacro)
@@ -5,18 +5,26 @@
   <xacro:property name="velocity" value="0.1"/>
   <xacro:macro name="leg" params="n xyz rpy parent">
-  <!--
-  <joint name="leg${n}-servo-joint" type="fixed">
+  <joint name="leg${n}_servo1_joint" type="fixed">
     <parent link="${parent}"/>
-    <child link="leg${n}-servo1"/>
-    <origin rpy="0 0 0" xyz="0 0 0"/>
+    <child link="leg${n}_servo1"/>
+    <origin xyz="${xyz}" rpy="${rpy}"/>
   </joint>
-  <xacro:lx224 name="leg${n}-servo1" rpy="0 0 0" xyz="0 0 0" color="red"/>
-  -->
+  <link name="leg${n}_servo1">
+    <visual>
+      <geometry>
+        <mesh filename="package://quaro_description/meshes/servo-hip.stl" scale="${scale} ${scale} ${scale}"/>
+      </geometry>
+      <origin xyz="0 0 0" rpy="0 0 0"/>
+      <material name="red">
+        <color rgba="1 0 0 1"/>
+      </material>
+    </visual>
+  </link>
   <!-- Leg Joint 1 -->
   <joint name="leg${n}_joint1" type="revolute">
-    <parent link="${parent}"/>
+    <parent link="leg${n}_servo1"/>
     <child link="leg${n}_link1"/>
-    <origin xyz="${xyz}" rpy="${rpy}"/>
-    <axis xyz="0 0 1"/>
+    <origin xyz="0 0 0" rpy="0 0 0"/>
+    <axis xyz="0 1 0"/>
     <limit effort="100.0" velocity="1.0" lower="-${2*pi/3}" upper="${2*pi/3}"/>
   </joint>
@@ -24,15 +32,17 @@
     <visual>
       <geometry>
-        <box size="0.1 0.4 0.1"/>
+        <mesh filename="package://quaro_description/meshes/hip.stl" scale="${scale} ${scale} ${scale}"/>
       </geometry>
-      <origin xyz="0.0 0.4 0.0" rpy="0 0 0"/>
+      <origin xyz="0 0 0" rpy="${pi/2} 0 ${pi/2}"/>
+      <material name="blue">
+        <color rgba="0 0 1 1"/>
+      </material>
     </visual>
   </link>
-  <!-- Leg Joint 2 -->
-  <joint name="leg${n}_joint2" type="revolute">
+  <joint name="leg${n}_servo2_joint" type="revolute">
     <parent link="leg${n}_link1"/>
     <child link="leg${n}_link2"/>
-    <origin xyz="0.0 0.6 0.0" rpy="0 0 0"/>
-    <axis xyz="0 0 1"/>
+    <origin xyz="0.04 0 0" rpy="-${pi/2} 0 ${pi}"/>
+    <axis xyz="0 1 0"/>
     <limit effort="100.0" velocity="1.0" lower="-${2*pi/3}" upper="${2*pi/3}"/>
   </joint>
@@ -40,15 +50,17 @@
     <visual>
       <geometry>
-        <box size="0.1 0.4 0.1"/>
+        <mesh filename="package://quaro_description/meshes/knee.stl" scale="${scale} ${scale} ${scale}"/>
       </geometry>
-      <origin xyz="0.0 0.4 0.0" rpy="0 0 0"/>
+      <origin xyz="0 0 0" rpy="0 0 0"/>
+      <material name="green">
+        <color rgba="0 1 0 1"/>
+      </material>
     </visual>
   </link>
-  <!-- Leg Joint 3 -->
-  <joint name="leg${n}_joint3" type="revolute">
+  <joint name="leg${n}_servo3_joint" type="revolute">
     <parent link="leg${n}_link2"/>
     <child link="leg${n}_link3"/>
-    <origin xyz="0.0 0.6 0.0" rpy="0 0 0"/>
-    <axis xyz="0 0 1"/>
+    <origin xyz="-0.054 0 0.015" rpy="${pi} 0 0"/>
+    <axis xyz="0 1 0"/>
     <limit effort="100.0" velocity="1.0" lower="-${2*pi/3}" upper="${2*pi/3}"/>
   </joint>
@@ -56,7 +68,10 @@
     <visual>
       <geometry>
-        <box size="0.1 0.4 0.1"/>
+        <mesh filename="package://quaro_description/meshes/shin.stl" scale="${scale} ${scale} ${scale}"/>
       </geometry>
-      <origin xyz="0.0 0.4 0.0" rpy="0 0 0"/>
+      <origin xyz="0 0 0" rpy="0 0 0"/>
+      <material name="grey">
+        <color rgba="0.5 0.5 0.5 1"/>
+      </material>
     </visual>
   </link>

File: src/quaro_description/urdf/quaro.xacro (robot description, xacro)
@@ -3,6 +3,4 @@
   <!-- Various constant definitions -->
   <xacro:include filename='$(find quaro_description)/urdf/common/constants.xacro'/>
-  <!-- Servo visual -->
-  <xacro:include filename="$(find quaro_description)/urdf/common/lx-224hv.xacro"/>
   <!-- Material Colors -->
   <xacro:include filename="$(find quaro_description)/urdf/common/colors.xacro"/>
@@ -13,12 +11,19 @@
     <visual>
       <geometry>
-        <cylinder radius="0.1" length="0.2"/>
+        <mesh filename="package://quaro_description/meshes/body.stl" scale="${scale} ${scale} ${scale}"/>
       </geometry>
-      <origin xyz="0 0 0" rpy="0 0 0"/>
+      <origin xyz="0 0 0" rpy="-${pi/2} 0 0"/>
+      <material name="grey">
+        <color rgba="0.5 0.5 0.5 1"/>
+      </material>
     </visual>
   </link>
-  <!-- Chain A -->
-  <xacro:leg n="1" parent="base_link" xyz="0.0 -0.4 0.0" rpy="${pi} 0 ${pi/4}"/>
-  <!-- Chain B -->
-  <xacro:leg n="2" parent="base_link" xyz="0.0 0.4 0.0" rpy="${pi} 0 ${3*pi/4}"/>
+  <!-- Chain 1 -->
+  <xacro:leg n="1" parent="base_link" xyz="0.0470 0.0920 0.0257" rpy="${pi/2} 0 ${pi/4}"/>
+  <!-- Chain 2 -->
+  <xacro:leg n="2" parent="base_link" xyz="-0.0470 0.0920 0.0257" rpy="${pi/2} 0 ${3*pi/4}"/>
+  <!-- Chain 3 -->
+  <xacro:leg n="3" parent="base_link" xyz="0.0470 -0.0920 0.0257" rpy="${pi/2} 0 -${pi/4}"/>
+  <!-- Chain 4 -->
+  <xacro:leg n="4" parent="base_link" xyz="-0.0470 -0.0920 0.0257" rpy="${pi/2} 0 -${3*pi/4}"/>
 </robot>
